Commit message: Fixup latest rviz, latest nav2, hardware changes, my fs changes.

File: openrover_demo/urdf/rover.urdf (robot description, URDF)
Before this commit: robot 2WD_rover_robotics, 11 links, 10 joints
Joints:
- joint lidar_link_joint: origin xyz=0 0 0.0488 rpy=0 0 0 -> xyz=0.10795 0 0.0635 rpy=0 0 0

File: openrover_demo/urdf/rover.urdf.xacro (robot description, xacro)
@@ -200,5 +200,5 @@
     <parent link="cpu_link"/>
     <child link="lidar_link"/>
-    <origin xyz="0 0 0.0488" rpy="0 0 0"/>
+    <origin xyz="0.10795 0 0.0635" rpy="0 0 0"/>
   </joint>
   <link name="lidar_link">

Commit message: Flip lidar around

File: openrover_demo/urdf/rover.urdf (robot description, URDF)
Before this commit: robot 2WD_rover_robotics, 11 links, 10 joints
Joints:
- joint lidar_link_joint: origin xyz=0.10795 0 0.0635 rpy=0 0 0 -> xyz=0.10795 0 0.0635 rpy=0 0 3.14

File: openrover_demo/urdf/rover.urdf.xacro (robot description, xacro)
@@ -200,5 +200,5 @@
     <parent link="cpu_link"/>
     <child link="lidar_link"/>
-    <origin xyz="0.10795 0 0.0635" rpy="0 0 0"/>
+    <origin xyz="0.10795 0 0.0635" rpy="0 0 3.14"/>
   </joint>
   <link name="lidar_link">
