Commit message: URDF updates for the openrover demo configuration
- Update masses based on real-world measurements
- Reset inertial values to a sane placeholder value
- Align topics and frequencies with actual robot configuration
- Remove camera from model

File: openrover_demo/urdf/2WD_Rover.gazebo.xacro (robot description, xacro)
@@ -2,5 +2,4 @@
 <robot name="rover_sim" xmlns:xacro="http://ros.org/wiki/xacro">
   <xacro:arg name="laser_visual"  default="false"/>
-  <xacro:arg name="camera_visual" default="false"/>
   <xacro:arg name="imu_visual"    default="false"/>
   <gazebo reference="base_link">
@@ -62,5 +61,5 @@
   </gazebo>
   <gazebo>
-    <plugin name="turtlebot3_waffle_controller" filename="libgazebo_ros_diff_drive.so">
+    <plugin name="openrover_controller" filename="libgazebo_ros_diff_drive.so">
       <commandTopic>cmd_vel</commandTopic>
       <odometryTopic>odom</odometryTopic>
@@ -71,7 +70,7 @@
       <publishWheelTF>false</publishWheelTF>
       <publishTf>true</publishTf>
-      <publishWheelJointState>true</publishWheelJointState>
+      <publishWheelJointState>false</publishWheelJointState>
       <legacyMode>false</legacyMode>
-      <updateRate>30</updateRate>
+      <updateRate>15</updateRate>
       <leftJoint>wheel_left_joint</leftJoint>
       <rightJoint>wheel_right_joint</rightJoint>
@@ -84,12 +83,18 @@
   </gazebo>
   <gazebo>
+    <plugin name="openrover_caster_publisher" filename="libgazebo_ros_joint_state_publisher.so">
+      <jointName>caster_back_left_joint,caster_back_right_joint,wheel_left_joint,wheel_right_joint</jointName>
+      <updateRate>15</updateRate>
+    </plugin>
+  </gazebo>
+  <gazebo>
     <plugin name="imu_plugin" filename="libgazebo_ros_imu.so">
       <alwaysOn>true</alwaysOn>
       <bodyName>imu_link</bodyName>
       <frameName>imu_link</frameName>
-      <topicName>imu</topicName>
+      <topicName>imu/data</topicName>
       <serviceName>imu_service</serviceName>
       <gaussianNoise>0.0</gaussianNoise>
-      <updateRate>200</updateRate>
+      <updateRate>20</updateRate>
       <imu>
         <noise>
@@ -116,5 +121,5 @@
       <pose>0 0 0 0 0 0</pose>
       <visualize>$(arg laser_visual)</visualize>
-      <update_rate>5</update_rate>
+      <update_rate>13</update_rate>
       <ray>
         <scan>
@@ -139,48 +144,5 @@
       <plugin name="gazebo_ros_lds_lfcd_controller" filename="libgazebo_ros_laser.so">
         <topicName>scan</topicName>
-        <frameName>base_scan</frameName>
-      </plugin>
-    </sensor>
-  </gazebo>
-  <gazebo reference="camera_rgb_frame">
-    <sensor type="depth" name="realsense_R200">
-      <always_on>true</always_on>
-      <visualize>$(arg camera_visual)</visualize>
-      <camera>
-          <horizontal_fov>1.3439</horizontal_fov>
-          <image>
-              <width>1920</width>
-              <height>1080</height>
-              <format>R8G8B8</format>
-          </image>
-          <depth_camera></depth_camera>
-          <clip>
-              <near>0.03</near>
-              <far>100</far>
-          </clip>
-      </camera>
-      <plugin name="camera_controller" filename="libgazebo_ros_openni_kinect.so">
-        <baseline>0.2</baseline>
-        <alwaysOn>true</alwaysOn>
-        <updateRate>30.0</updateRate>
-        <cameraName>camera</cameraName>
-        <frameName>camera_rgb_optical_frame</frameName>
-        <imageTopicName>rgb/image_raw</imageTopicName>
-        <depthImageTopicName>depth/image_raw</depthImageTopicName>
-        <pointCloudTopicName>depth/points</pointCloudTopicName>
-        <cameraInfoTopicName>rgb/camera_info</cameraInfoTopicName>
-        <depthImageCameraInfoTopicName>depth/camera_info</depthImageCameraInfoTopicName>
-        <pointCloudCutoff>0.4</pointCloudCutoff>
-            <hackBaseline>0.07</hackBaseline>
-            <distortionK1>0.0</distortionK1>
-            <distortionK2>0.0</distortionK2>
-            <distortionK3>0.0</distortionK3>
-            <distortionT1>0.0</distortionT1>
-            <distortionT2>0.0</distortionT2>
-        <CxPrime>0.0</CxPrime>
-        <Cx>0.0</Cx>
-        <Cy>0.0</Cy>
-        <focalLength>0</focalLength>
-        <hackBaseline>0</hackBaseline>
+        <frameName>lidar_link</frameName>
       </plugin>
     </sensor>

File: openrover_demo/urdf/rover.urdf (robot description, URDF)
Before this commit: robot 2WD_rover_robotics, 11 links, 10 joints
Links:
- link base_link: mass 1.3729096e+00 -> 7.5
- link caster_back_left_link: mass 0.005 -> 0.6
- link caster_back_right_link: mass 0.005 -> 0.6
- link cpu_link: mass None -> 0.640
- link imu_link: mass None -> 0.04
- link lidar_link: mass None -> 0.220
- link plate_link: mass None -> 0.65
- link sheetmetal_link: mass None -> 0.6
- link wheel_left_link: mass 2.8498940e-02 -> 1.525
- link wheel_right_link: mass 2.8498940e-02 -> 1.525

File: openrover_demo/urdf/rover.urdf.xacro (robot description, xacro)
@@ -6,5 +6,5 @@
   <joint name="base_joint" type="fixed">
     <parent link="base_footprint"/>
-    <child link="base_link" />
+    <child link="base_link"/>
     <origin xyz="0 0 0.12" rpy="0 0 0"/>
   </joint>
@@ -24,9 +24,9 @@
     </collision>
     <inertial>
-      <origin xyz="0 0 0" rpy="0 0 0"/>
-      <mass value="1.3729096e+00"/>
-      <inertia ixx="8.7002718e-03" ixy="-4.7576583e-05" ixz="1.1160499e-04"
-               iyy="8.6195418e-03" iyz="-3.5422299e-06"
-               izz="1.4612727e-02" />
+      <origin xyz="0 0 0" rpy="0 0 0" />
+      <mass value="7.5" />
+      <inertia ixx="0.001" ixy="0.0" ixz="0.0"
+               iyy="0.001" iyz="0.0"
+               izz="0.001" />
     </inertial>
   </link>
@@ -53,9 +53,9 @@
     <inertial>
       <origin xyz="0 0 0" />
-      <mass value="2.8498940e-02" />
-      <inertia ixx="1.1175580e-05" ixy="-4.2369783e-11" ixz="-5.9381719e-09"
-               iyy="1.1192413e-05" iyz="-1.4400107e-11"
-               izz="2.0712558e-05" />
-      </inertial>
+      <mass value="1.525" />
+      <inertia ixx="0.001" ixy="0.0" ixz="0.0"
+               iyy="0.001" iyz="0.0"
+               izz="0.001" />
+    </inertial>
   </link>
   <joint name="wheel_right_joint" type="continuous">
@@ -81,8 +81,8 @@
     <inertial>
       <origin xyz="0 0 0" />
-      <mass value="2.8498940e-02" />
-      <inertia ixx="1.1175580e-05" ixy="-4.2369783e-11" ixz="-5.9381719e-09"
-               iyy="1.1192413e-05" iyz="-1.4400107e-11"
-               izz="2.0712558e-05" />
+      <mass value="1.525" />
+      <inertia ixx="0.001" ixy="0.0" ixz="0.0"
+               iyy="0.001" iyz="0.0"
+               izz="0.001" />
     </inertial>
   </link>
@@ -106,4 +106,11 @@
       </geometry>
     </collision>
+    <inertial>
+      <origin xyz="0 0 0" />
+      <mass value="0.6" />
+      <inertia ixx="0.001" ixy="0.0" ixz="0.0"
+               iyy="0.001" iyz="0.0"
+               izz="0.001" />
+    </inertial>
   </link>
   <joint name="plate_link_joint" type="fixed">
@@ -120,4 +127,11 @@
       <material name="light_black"/>
     </visual>
+    <inertial>
+      <origin xyz="0 0 0" />
+      <mass value="0.65" />
+      <inertia ixx="0.001" ixy="0.0" ixz="0.0"
+               iyy="0.001" iyz="0.0"
+               izz="0.001" />
+    </inertial>
   </link>
   <joint name="imu_link_joint" type="fixed">
@@ -134,4 +148,11 @@
       <material name="light_black"/>
     </visual>
+    <inertial>
+      <origin xyz="0 0 0" />
+      <mass value="0.04" />
+      <inertia ixx="0.001" ixy="0.0" ixz="0.0"
+               iyy="0.001" iyz="0.0"
+               izz="0.001" />
+    </inertial>
   </link>
   <joint name="cpu_link_joint" type="fixed">
@@ -148,4 +169,11 @@
       <material name="light_black"/>
     </visual>
+    <inertial>
+      <origin xyz="0 0 0" />
+      <mass value="0.640" />
+      <inertia ixx="0.001" ixy="0.0" ixz="0.0"
+               iyy="0.001" iyz="0.0"
+               izz="0.001" />
+    </inertial>
   </link>
   <joint name="lidar_link_joint" type="fixed">
@@ -162,4 +190,11 @@
       <material name="light_black"/>
     </visual>
+    <inertial>
+      <origin xyz="0 0 0" />
+      <mass value="0.220" />
+      <inertia ixx="0.001" ixy="0.0" ixz="0.0"
+               iyy="0.001" iyz="0.0"
+               izz="0.001" />
+    </inertial>
   </link>
   <joint name="caster_back_right_joint" type="continuous">
@@ -185,5 +220,5 @@
     <inertial>
       <origin xyz="0 0 0" />
-      <mass value="0.005" />
+      <mass value="0.6" />
       <inertia ixx="0.001" ixy="0.0" ixz="0.0"
                iyy="0.001" iyz="0.0"
@@ -213,5 +248,5 @@
     <inertial>
       <origin xyz="0 0 0" />
-      <mass value="0.005" />
+      <mass value="0.6" />
       <inertia ixx="0.001" ixy="0.0" ixz="0.0"
                iyy="0.001" iyz="0.0"

Commit message: More robot description updates
- Real values for inertia
- Some slightly more interesting colors
- Tweaks to the gazebo data to better approximate hardware

File: openrover_demo/urdf/2WD_Rover.gazebo.xacro (robot description, xacro)
@@ -35,5 +35,5 @@
     <material>Gazebo/White</material>
   </gazebo>
-  <gazebo reference="caster_back_right_link">
+  <gazebo reference="caster_back_left_link">
     <mu1>0.1</mu1>
     <mu2>0.1</mu2>
@@ -44,5 +44,5 @@
     <material>Gazebo/FlatBlack</material>
   </gazebo>
-  <gazebo reference="caster_back_left_link">
+  <gazebo reference="caster_back_right_link">
     <mu1>0.1</mu1>
     <mu2>0.1</mu2>
@@ -66,11 +66,11 @@
       <odometryFrame>odom</odometryFrame>
       <odometrySource>world</odometrySource>
-      <publishOdomTF>true</publishOdomTF>
+      <publishOdomTF>false</publishOdomTF>
       <robotBaseFrame>base_footprint</robotBaseFrame>
       <publishWheelTF>false</publishWheelTF>
-      <publishTf>true</publishTf>
+      <publishTf>false</publishTf>
       <publishWheelJointState>false</publishWheelJointState>
       <legacyMode>false</legacyMode>
-      <updateRate>15</updateRate>
+      <updateRate>10</updateRate>
       <leftJoint>wheel_left_joint</leftJoint>
       <rightJoint>wheel_right_joint</rightJoint>
@@ -84,6 +84,6 @@
   <gazebo>
     <plugin name="openrover_caster_publisher" filename="libgazebo_ros_joint_state_publisher.so">
-      <jointName>caster_back_left_joint,caster_back_right_joint,wheel_left_joint,wheel_right_joint</jointName>
-      <updateRate>15</updateRate>
+      <jointName>wheel_left_joint,wheel_right_joint,caster_back_left_joint,caster_back_right_joint</jointName>
+      <updateRate>30</updateRate>
     </plugin>
   </gazebo>
@@ -96,5 +96,5 @@
       <serviceName>imu_service</serviceName>
       <gaussianNoise>0.0</gaussianNoise>
-      <updateRate>20</updateRate>
+      <updateRate>30</updateRate>
       <imu>
         <noise>
@@ -142,5 +142,5 @@
         </noise>
       </ray>
-      <plugin name="gazebo_ros_lds_lfcd_controller" filename="libgazebo_ros_laser.so">
+      <plugin name="gazebo_ros_lds_lfcd_controller" filename="libgazebo_ros_gpu_laser.so">
         <topicName>scan</topicName>
         <frameName>lidar_link</frameName>

File: openrover_demo/urdf/common_properties.xacro (robot description, xacro)
@@ -32,3 +32,6 @@
     <color rgba="1.0 1.0 1.0 1.0"/>
   </material>
+  <material name="acrylic">
+    <color rgba="0.9 0.9 1.0 0.6"/>
+  </material>
 </robot>

File: openrover_demo/urdf/rover.urdf (robot description, URDF)
Before this commit: robot 2WD_rover_robotics, 11 links, 10 joints
Links:
- link caster_back_left_link: mass 0.6 -> 0.41
- link caster_back_right_link: mass 0.6 -> 0.41
- link cpu_link: mass 0.640 -> 0.64
- link sheetmetal_link: geometry collision box size=0.065 0.4 0.008; visual mesh filename=package://openrover_demo/meshes/sheetmetal_part.stl scale=1 1 1
Joints:
- joint caster_back_left_joint: origin xyz=-0.36 0.17 -0.01 rpy=0 0 0 -> xyz=-0.01 0.17 -0.01 rpy=0 0 0; parent base_link -> sheetmetal_link
- joint caster_back_right_joint: origin xyz=-0.36 -0.17 -0.01 rpy=0 0 0 -> xyz=-0.01 -0.17 -0.01 rpy=0 0 0; parent base_link -> sheetmetal_link

File: openrover_demo/urdf/rover.urdf.xacro (robot description, xacro)
@@ -14,19 +14,24 @@
       <geometry>
         <mesh filename="package://openrover_demo/meshes/2WD_OpenRover.stl" scale="1 1 1"/>
-      </geometry>
-      <material name="light_black"/>
-    </visual>
-    <collision>
-      <origin xyz="-0.14 0 0" rpy="0 0 0"/>
+      <!--
+      <origin xyz="-0.142 0 0" rpy="0 0 0"/>
       <geometry>
         <box size="0.42 0.25 0.12"/>
-      </geometry>
-    </collision>
-    <inertial>
-      <origin xyz="0 0 0" rpy="0 0 0" />
+        -->
+      </geometry>
+      <material name="dark"/>
+    </visual>
+    <collision>
+      <origin xyz="-0.142 0 0" rpy="0 0 0"/>
+      <geometry>
+        <box size="0.42 0.25 0.12"/>
+      </geometry>
+    </collision>
+    <inertial>
+      <origin xyz="-0.142 0 0" rpy="0 0 0" />
       <mass value="7.5" />
-      <inertia ixx="0.001" ixy="0.0" ixz="0.0"
-               iyy="0.001" iyz="0.0"
-               izz="0.001" />
+      <inertia ixx="4.806e-2"
+               ixy="0.0" iyy="1.193e-1"
+               ixz="0.0" iyz="0.0" izz="1.493e-1" />
     </inertial>
   </link>
@@ -42,19 +47,24 @@
       <geometry>
         <mesh filename="package://openrover_demo/meshes/left_wheel.stl" scale="1 1 1"/>
-      </geometry>
-      <material name="light_black"/>
-    </visual>
-    <collision>
-      <origin xyz="0 0 0" rpy="0 0 0"/>
-      <geometry>
-        <cylinder length="0.07" radius="0.12"/>
-      </geometry>
-    </collision>
-    <inertial>
-      <origin xyz="0 0 0" />
+      <!--
+      <origin xyz="0 0 0" rpy="0 0 3.14"/>
+      <geometry>
+        <cylinder length="0.07" radius="0.12"/>
+        -->
+      </geometry>
+      <material name="black"/>
+    </visual>
+    <collision>
+      <origin xyz="0 0 0" rpy="0 0 3.14"/>
+      <geometry>
+        <cylinder length="0.07" radius="0.12"/>
+      </geometry>
+    </collision>
+    <inertial>
+      <origin xyz="0 0 0" rpy="0 0 3.14" />
       <mass value="1.525" />
-      <inertia ixx="0.001" ixy="0.0" ixz="0.0"
-               iyy="0.001" iyz="0.0"
-               izz="0.001" />
+      <inertia ixx="6.723e-3"
+               ixy="0.0" iyy="6.723e-3"
+               ixz="0.0" iyz="0.0" izz="1.220e-2" />
     </inertial>
   </link>
@@ -70,19 +80,24 @@
       <geometry>
         <mesh filename="package://openrover_demo/meshes/right_wheel.stl" scale="1 1 1"/>
-      </geometry>
-      <material name="light_black"/>
-    </visual>
-    <collision>
-      <origin xyz="0 0 0" rpy="0 0 0"/>
-      <geometry>
-        <cylinder length="0.07" radius="0.12"/>
-      </geometry>
-    </collision>
-    <inertial>
-      <origin xyz="0 0 0" />
+      <!--
+      <origin xyz="0 0 0" rpy="0 0 0"/>
+      <geometry>
+        <cylinder length="0.07" radius="0.12"/>
+        -->
+      </geometry>
+      <material name="black"/>
+    </visual>
+    <collision>
+      <origin xyz="0 0 0" rpy="0 0 0"/>
+      <geometry>
+        <cylinder length="0.07" radius="0.12"/>
+      </geometry>
+    </collision>
+    <inertial>
+      <origin xyz="0 0 0" rpy="0 0 0" />
       <mass value="1.525" />
-      <inertia ixx="0.001" ixy="0.0" ixz="0.0"
-               iyy="0.001" iyz="0.0"
-               izz="0.001" />
+      <inertia ixx="6.723e-3"
+               ixy="0.0" iyy="6.723e-3"
+               ixz="0.0" iyz="0.0" izz="1.220e-2" />
     </inertial>
   </link>
@@ -97,11 +112,16 @@
       <geometry>
         <mesh filename="package://openrover_demo/meshes/sheetmetal_part.stl" scale="1 1 1"/>
-      </geometry>
-      <material name="light_black"/>
-    </visual>
-    <collision>
-      <origin xyz="-0.05 0 0" rpy="0 0 0"/>
-      <geometry>
-        <box size="0.065 0.3 0.008"/>
+      <!--
+      <origin xyz="0 0 0" rpy="0 0 0"/>
+      <geometry>
+        <box size="0.065 0.4 0.008"/>
+        -->
+      </geometry>
+      <material name="dark"/>
+    </visual>
+    <collision>
+      <origin xyz="-0.007 0 0" rpy="0 0 0"/>
+      <geometry>
+        <box size="0.065 0.4 0.008"/>
       </geometry>
     </collision>
@@ -109,7 +129,7 @@
       <origin xyz="0 0 0" />
       <mass value="0.6" />
-      <inertia ixx="0.001" ixy="0.0" ixz="0.0"
-               iyy="0.001" iyz="0.0"
-               izz="0.001" />
+      <inertia ixx="8.020e-3"
+               ixy="0.0" iyy="2.313e-4"
+               ixz="0.0" iyz="0.0" izz="8.211e-3" />
     </inertial>
   </link>
@@ -125,12 +145,12 @@
         <box size="0.381 0.254 0.005"/>
       </geometry>
-      <material name="light_black"/>
+      <material name="acrylic"/>
     </visual>
     <inertial>
       <origin xyz="0 0 0" />
       <mass value="0.65" />
-      <inertia ixx="0.001" ixy="0.0" ixz="0.0"
-               iyy="0.001" iyz="0.0"
-               izz="0.001" />
+      <inertia ixx="3.496e-3"
+               ixy="0.0" iyy="7.864e-3"
+               ixz="0.0" iyz="0.0" izz="1.136e-2" />
     </inertial>
   </link>
@@ -146,12 +166,12 @@
         <box size="0.01 0.01 0.002"/>
       </geometry>
-      <material name="light_black"/>
+      <material name="blue"/>
     </visual>
     <inertial>
       <origin xyz="0 0 0" />
       <mass value="0.04" />
-      <inertia ixx="0.001" ixy="0.0" ixz="0.0"
-               iyy="0.001" iyz="0.0"
-               izz="0.001" />
+      <inertia ixx="3.467e-7"
+               ixy="0.0" iyy="3.467e-7"
+               ixz="0.0" iyz="0.0" izz="6.667e-7" />
     </inertial>
   </link>
@@ -171,8 +191,8 @@
     <inertial>
       <origin xyz="0 0 0" />
-      <mass value="0.640" />
-      <inertia ixx="0.001" ixy="0.0" ixz="0.0"
-               iyy="0.001" iyz="0.0"
-               izz="0.001" />
+      <mass value="0.64" />
+      <inertia ixx="8.634e-4"
+               ixy="0.0" iyy="7.905e-4"
+               ixz="0.0" iyz="0.0" izz="1.387e-3" />
     </inertial>
   </link>
@@ -193,13 +213,46 @@
       <origin xyz="0 0 0" />
       <mass value="0.220" />
-      <inertia ixx="0.001" ixy="0.0" ixz="0.0"
-               iyy="0.001" iyz="0.0"
-               izz="0.001" />
+      <inertia ixx="1.214e-4"
+	       ixy="0.0" iyy="1.214e-4"
+               ixz="0.0" iyz="0.0" izz="1.597e-4" />
+    </inertial>
+  </link>
+  <joint name="caster_back_left_joint" type="continuous">
+    <parent link="sheetmetal_link"/>
+    <child link="caster_back_left_link"/>
+    <origin xyz="-0.01 0.17 -0.01" rpy="0 0 0"/>
+    <axis xyz="0 0 1"/>
+  </joint>
+  <link name="caster_back_left_link">
+    <visual>
+      <origin xyz="0 0 0" rpy="1.57 0 3.14"/>
+      <geometry>
+        <mesh filename="package://openrover_demo/meshes/left_caster_wheel.stl" scale="1 1 1"/>
+      <!--
+      <origin xyz="-0.028 0 -0.065" rpy="1.57 0 3.14"/>
+      <geometry>
+        <cylinder length="0.035" radius="0.048"/>
+        -->
+      </geometry>
+      <material name="grey"/>
+    </visual>
+    <collision>
+      <origin xyz="-0.028 0 -0.065" rpy="1.57 0 3.14"/>
+      <geometry>
+        <cylinder length="0.035" radius="0.048"/>
+      </geometry>
+    </collision>
+    <inertial>
+      <origin xyz="-0.005 0 -0.03" />
+      <mass value="0.41" />
+      <inertia ixx="3.841e-4"
+               ixy="0.0" iyy="4.592e-4"
+               ixz="0.0" iyz="0.0" izz="2.135e-4" />
     </inertial>
   </link>
   <joint name="caster_back_right_joint" type="continuous">
-    <parent link="base_link"/>
+    <parent link="sheetmetal_link"/>
     <child link="caster_back_right_link"/>
-    <origin xyz="-0.36 -0.17 -0.01" rpy="0 0 0"/>
+    <origin xyz="-0.01 -0.17 -0.01" rpy="0 0 0"/>
     <axis xyz="0 0 1"/>
   </joint>
@@ -209,47 +262,24 @@
       <geometry>
         <mesh filename="package://openrover_demo/meshes/right_caster_wheel.stl" scale="1 1 1"/>
-      </geometry>
-      <material name="light_black"/>
-    </visual>
-    <collision>
-      <origin xyz="-0.028 0 -0.065" rpy="1.57 0 0"/>
-      <geometry>
-        <cylinder length="0.035" radius="0.048"/>
-      </geometry>
-    </collision>
-    <inertial>
-      <origin xyz="0 0 0" />
-      <mass value="0.6" />
-      <inertia ixx="0.001" ixy="0.0" ixz="0.0"
-               iyy="0.001" iyz="0.0"
-               izz="0.001" />
-    </inertial>
-  </link>
-  <joint name="caster_back_left_joint" type="continuous">
-    <parent link="base_link"/>
-    <child link="caster_back_left_link"/>
-    <origin xyz="-0.36 0.17 -0.01" rpy="0 0 0"/>
-    <axis xyz="0 0 1"/>
-  </joint>
-  <link name="caster_back_left_link">
-    <visual>
-      <origin xyz="0 0 0" rpy="1.57 0 3.14"/>
-      <geometry>
-        <mesh filename="package://openrover_demo/meshes/left_caster_wheel.stl" scale="1 1 1"/>
-      </geometry>
-      <material name="light_black"/>
-    </visual>
-    <collision>
-      <origin xyz="-0.028 0 -0.065" rpy="1.57 0 0"/>
-      <geometry>
-        <cylinder length="0.035" radius="0.048"/>
-      </geometry>
-    </collision>
-    <inertial>
-      <origin xyz="0 0 0" />
-      <mass value="0.6" />
-      <inertia ixx="0.001" ixy="0.0" ixz="0.0"
-               iyy="0.001" iyz="0.0"
-               izz="0.001" />
+      <!--
+      <origin xyz="-0.028 0 -0.065" rpy="1.57 0 3.14"/>
+      <geometry>
+        <cylinder length="0.035" radius="0.048"/>
+        -->
+      </geometry>
+      <material name="grey"/>
+    </visual>
+    <collision>
+      <origin xyz="-0.028 0 -0.065" rpy="1.57 0 3.14"/>
+      <geometry>
+        <cylinder length="0.035" radius="0.048"/>
+      </geometry>
+    </collision>
+    <inertial>
+      <origin xyz="-0.005 0 -0.03" />
+      <mass value="0.41" />
+      <inertia ixx="3.841e-4"
+               ixy="0.0" iyy="4.592e-4"
+               ixz="0.0" iyz="0.0" izz="2.135e-4" />
     </inertial>
   </link>
