Commit message: Updates needed for simulation to work
- The model has been updated (mainly physics)
- The Gazebo part of the model now targets ROS2
- I included `urdf_spawner.py` because `spawn_model` isn't in gazebo_ros
  yet.

File: openrover_demo/urdf/2WD_Rover.gazebo.xacro (robot description, xacro)
@@ -1,125 +1,107 @@
 <?xml version="1.0"?>
 <robot name="rover_sim" xmlns:xacro="http://ros.org/wiki/xacro">
-  <xacro:arg name="laser_visual"  default="false"/>
-  <xacro:arg name="imu_visual"    default="false"/>
   <gazebo reference="base_link">
-    <material>Gazebo/DarkGrey</material>
+    <material>Gazebo/FlatBlack</material>
+  </gazebo>
+  <gazebo reference="sheetmetal_link">
+    <material>Gazebo/FlatBlack</material>
   </gazebo>
   <gazebo reference="wheel_left_link">
-    <mu1>0.1</mu1>
-    <mu2>0.1</mu2>
-    <kp>500000.0</kp>
-    <kd>10.0</kd>
-    <minDepth>0.001</minDepth>
-    <maxVel>0.1</maxVel>
-    <fdir1>1 0 0</fdir1>
-    <material>Gazebo/White</material>
+    <mu1>0.7</mu1>
+    <mu2>1.0</mu2>
+    <kp>300000.0</kp>
+    <material>Gazebo/Black</material>
   </gazebo>
   <gazebo reference="wheel_right_link">
-    <mu1>0.1</mu1>
-    <mu2>0.1</mu2>
-    <kp>500000.0</kp>
-    <kd>10.0</kd>
-    <minDepth>0.001</minDepth>
-    <maxVel>0.1</maxVel>
-    <fdir1>1 0 0</fdir1>
-    <material>Gazebo/White</material>
-  </gazebo>
-  <gazebo reference="sheetmetal_link">
-    <mu1>0.1</mu1>
-    <mu2>0.1</mu2>
-    <kp>1000000.0</kp>
-    <kd>100.0</kd>
-    <minDepth>0.001</minDepth>
-    <maxVel>1.0</maxVel>
-    <material>Gazebo/White</material>
+    <mu1>0.7</mu1>
+    <mu2>1.0</mu2>
+    <kp>300000.0</kp>
+    <material>Gazebo/Black</material>
   </gazebo>
   <gazebo reference="caster_back_left_link">
     <mu1>0.1</mu1>
-    <mu2>0.1</mu2>
-    <kp>1000000.0</kp>
-    <kd>100.0</kd>
-    <minDepth>0.001</minDepth>
-    <maxVel>1.0</maxVel>
-    <material>Gazebo/FlatBlack</material>
+    <mu2>0.6</mu2>
+    <kp>200000.0</kp>
+    <material>Gazebo/Grey</material>
   </gazebo>
   <gazebo reference="caster_back_right_link">
     <mu1>0.1</mu1>
-    <mu2>0.1</mu2>
-    <kp>1000000.0</kp>
-    <kd>100.0</kd>
-    <minDepth>0.001</minDepth>
-    <maxVel>1.0</maxVel>
-    <material>Gazebo/FlatBlack</material>
+    <mu2>0.6</mu2>
+    <kp>200000.0</kp>
+    <material>Gazebo/Grey</material>
+  </gazebo>
+  <gazebo reference="plate_link">
+    <material>Gazebo/GreyTransparent</material>
   </gazebo>
   <gazebo reference="imu_link">
-    <sensor type="imu" name="imu">
+    <sensor name="gazebo_imu" type="imu">
       <always_on>true</always_on>
-      <visualize>$(arg imu_visual)</visualize>
+      <update_rate>30.0</update_rate>
+      <plugin name="gazebo_imu" filename="libgazebo_ros_imu_sensor.so">
+        <ros>
+          <namespace>/imu</namespace>
+          <argument>~/out:=data</argument>
+        </ros>
+        <frame_name>imu_link</frame_name>
+      </plugin>
+      <imu>
+        <angular_velocity>
+          <x>
+            <noise type="gaussian">
+              <mean>0.0</mean>
+              <stddev>0.0052</stddev>
+            </noise>
+          </x>
+          <y>
+            <noise type="gaussian">
+              <mean>0.0</mean>
+              <stddev>0.0052</stddev>
+            </noise>
+          </y>
+          <z>
+            <noise type="gaussian">
+              <mean>0.0</mean>
+              <stddev>0.0052</stddev>
+            </noise>
+          </z>
+        </angular_velocity>
+        <linear_acceleration>
+          <x>
+            <noise type="gaussian">
+              <mean>0.0</mean>
+              <stddev>0.0015</stddev>
+            </noise>
+          </x>
+          <y>
+            <noise type="gaussian">
+              <mean>0.0</mean>
+              <stddev>0.0015</stddev>
+            </noise>
+          </y>
+          <z>
+            <noise type="gaussian">
+              <mean>0.0</mean>
+              <stddev>0.0015</stddev>
+            </noise>
+          </z>
+        </linear_acceleration>
+      </imu>
     </sensor>
-    <material>Gazebo/Grey</material>
+    <material>Gazebo/Blue</material>
   </gazebo>
-  <gazebo>
-    <plugin name="openrover_controller" filename="libgazebo_ros_diff_drive.so">
-      <commandTopic>cmd_vel</commandTopic>
-      <odometryTopic>odom</odometryTopic>
-      <odometryFrame>odom</odometryFrame>
-      <odometrySource>world</odometrySource>
-      <publishOdomTF>false</publishOdomTF>
-      <robotBaseFrame>base_footprint</robotBaseFrame>
-      <publishWheelTF>false</publishWheelTF>
-      <publishTf>false</publishTf>
-      <publishWheelJointState>false</publishWheelJointState>
-      <legacyMode>false</legacyMode>
-      <updateRate>10</updateRate>
-      <leftJoint>wheel_left_joint</leftJoint>
-      <rightJoint>wheel_right_joint</rightJoint>
-      <wheelSeparation>0.287</wheelSeparation>
-      <wheelDiameter>0.066</wheelDiameter>
-      <wheelAcceleration>1</wheelAcceleration>
-      <wheelTorque>10</wheelTorque>
-      <rosDebugLevel>na</rosDebugLevel>
-    </plugin>
+  <gazebo reference="cpu_link">
+    <material>Gazebo/DarkGrey</material>
   </gazebo>
-  <gazebo>
-    <plugin name="openrover_caster_publisher" filename="libgazebo_ros_joint_state_publisher.so">
-      <jointName>wheel_left_joint,wheel_right_joint,caster_back_left_joint,caster_back_right_joint</jointName>
-      <updateRate>30</updateRate>
-    </plugin>
-  </gazebo>
-  <gazebo>
-    <plugin name="imu_plugin" filename="libgazebo_ros_imu.so">
-      <alwaysOn>true</alwaysOn>
-      <bodyName>imu_link</bodyName>
-      <frameName>imu_link</frameName>
-      <topicName>imu/data</topicName>
-      <serviceName>imu_service</serviceName>
-      <gaussianNoise>0.0</gaussianNoise>
-      <updateRate>30</updateRate>
-      <imu>
-        <noise>
-          <type>gaussian</type>
-          <rate>
-            <mean>0.0</mean>
-            <stddev>2e-4</stddev>
-            <bias_mean>0.0000075</bias_mean>
-            <bias_stddev>0.0000008</bias_stddev>
-          </rate>
-          <accel>
-            <mean>0.0</mean>
-            <stddev>1.7e-2</stddev>
-            <bias_mean>0.1</bias_mean>
-            <bias_stddev>0.001</bias_stddev>
-          </accel>
-        </noise>
-      </imu>
-    </plugin>
-  </gazebo>
-  <gazebo reference="base_scan">
-    <material>Gazebo/FlatBlack</material>
-    <sensor type="ray" name="lds_lfcd_sensor">
-      <pose>0 0 0 0 0 0</pose>
-      <visualize>$(arg laser_visual)</visualize>
-      <update_rate>13</update_rate>
+  <gazebo reference="lidar_link">
+    <sensor name="gazebo_lidar" type="ray">
+      <update_rate>12.0</update_rate>
+      <plugin name="gazebo_lidar" filename="libgazebo_ros_ray_sensor.so">
+        <ros>
+          <argument>~/out:=scan</argument>
+          <namespace></namespace>
+        </ros>
+        <output_type>sensor_msgs/LaserScan</output_type>
+        <frame_name>lidar_link</frame_name>
+      </plugin>
       <ray>
         <scan>
@@ -127,6 +109,6 @@
             <samples>360</samples>
             <resolution>1</resolution>
-            <min_angle>0.0</min_angle>
-            <max_angle>6.28319</max_angle>
+            <min_angle>-3.14159</min_angle>
+            <max_angle>3.14159</max_angle>
           </horizontal>
         </scan>
@@ -142,9 +124,34 @@
         </noise>
       </ray>
-      <plugin name="gazebo_ros_lds_lfcd_controller" filename="libgazebo_ros_gpu_laser.so">
-        <topicName>scan</topicName>
-        <frameName>lidar_link</frameName>
-      </plugin>
     </sensor>
+    <material>Gazebo/DarkGrey</material>
+  </gazebo>
+  <gazebo>
+    <plugin name="gazebo_base_controller" filename="libgazebo_ros_diff_drive.so">
+      <odometry_frame>odom</odometry_frame>
+      <publish_odom>true</publish_odom>
+      <publish_odom_tf>false</publish_odom_tf>
+      <robot_base_frame>base_footprint</robot_base_frame>
+      <publish_wheel_tf>false</publish_wheel_tf>
+      <update_rate>15.0</update_rate>
+      <left_joint>wheel_left_joint</left_joint>
+      <right_joint>wheel_right_joint</right_joint>
+      <wheel_separation>0.358</wheel_separation>
+      <wheel_diameter>0.24</wheel_diameter>
+      <max_wheel_acceleration>0.7</max_wheel_acceleration>
+      <max_wheel_torque>8</max_wheel_torque>
+      <ros>
+        <argument>odom:=odom_raw</argument>
+      </ros>
+    </plugin>
+  </gazebo>
+  <gazebo>
+    <plugin name="gazebo_joint_publisher" filename="libgazebo_ros_joint_state_publisher.so">
+      <joint_name>wheel_left_joint</joint_name>
+      <joint_name>wheel_right_joint</joint_name>
+      <joint_name>caster_back_left_joint</joint_name>
+      <joint_name>caster_back_right_joint</joint_name>
+      <update_rate>30.0</update_rate>
+    </plugin>
   </gazebo>
 </robot>

File: openrover_demo/urdf/rover.urdf (robot description, URDF)
Before this commit: robot 2WD_rover_robotics, 11 links, 10 joints
Links:
- link caster_back_left_link: geometry collision cylinder length=0.0035 radius=0.05; visual mesh filename=package://openrover_demo/meshes/left_caster_wheel.stl scale=1 1 1
- link caster_back_right_link: geometry collision cylinder length=0.0035 radius=0.05; visual mesh filename=package://openrover_demo/meshes/right_caster_wheel.stl scale=1 1 1

File: openrover_demo/urdf/rover.urdf.xacro (robot description, xacro)
@@ -214,5 +214,5 @@
       <mass value="0.220" />
       <inertia ixx="1.214e-4"
-	       ixy="0.0" iyy="1.214e-4"
+               ixy="0.0" iyy="1.214e-4"
                ixz="0.0" iyz="0.0" izz="1.597e-4" />
     </inertial>
@@ -223,4 +223,5 @@
     <origin xyz="-0.01 0.17 -0.01" rpy="0 0 0"/>
     <axis xyz="0 0 1"/>
+    <dynamics damping="0.1" friction="0.01"/>
   </joint>
   <link name="caster_back_left_link">
@@ -238,7 +239,7 @@
     </visual>
     <collision>
-      <origin xyz="-0.028 0 -0.065" rpy="1.57 0 3.14"/>
-      <geometry>
-        <cylinder length="0.035" radius="0.048"/>
+      <origin xyz="-0.035 0 -0.065" rpy="1.57 0 3.14"/>
+      <geometry>
+        <cylinder length="0.0035" radius="0.05"/>
       </geometry>
     </collision>
@@ -256,4 +257,5 @@
     <origin xyz="-0.01 -0.17 -0.01" rpy="0 0 0"/>
     <axis xyz="0 0 1"/>
+    <dynamics damping="0.1" friction="0.01"/>
   </joint>
   <link name="caster_back_right_link">
@@ -271,7 +273,7 @@
     </visual>
     <collision>
-      <origin xyz="-0.028 0 -0.065" rpy="1.57 0 3.14"/>
-      <geometry>
-        <cylinder length="0.035" radius="0.048"/>
+      <origin xyz="-0.035 0 -0.065" rpy="1.57 0 3.14"/>
+      <geometry>
+        <cylinder length="0.0035" radius="0.05"/>
       </geometry>
     </collision>

Commit message: fix launch files and urdf

File: openrover_demo/urdf/2WD_Rover.gazebo.xacro (robot description, xacro)
@@ -142,5 +142,5 @@
       <max_wheel_torque>8</max_wheel_torque>
       <ros>
-        <argument>odom:=odom_raw</argument>
+        <argument>odom:=odom</argument>
       </ros>
     </plugin>

File: openrover_demo/urdf/rover.urdf (robot description, URDF)
Before this commit: robot 2WD_rover_robotics, 11 links, 10 joints
Links:
- added link camera_link, mass 0.220; visual cylinder length=0.0476 radius=0.0381
Joints:
- added joint camera_link_joint: type fixed, parent cpu_link, child camera_link, origin xyz=0.10795 0 0.0635 rpy=0 0 3.14

File: openrover_demo/urdf/rover.urdf.xacro (robot description, xacro)
@@ -6,5 +6,5 @@
   <joint name="base_joint" type="fixed">
     <parent link="base_footprint"/>
-    <child link="base_link"/>
+    <child link="base"/>
     <origin xyz="0 0 0.12" rpy="0 0 0"/>
   </joint>
@@ -286,3 +286,24 @@
     </inertial>
   </link>
+<joint name="camera_link_joint" type="fixed">
+    <parent link="cpu_link"/>
+    <child link="camera_link"/>
+    <origin xyz="0.10795 0 0.0635" rpy="0 0 3.14"/>
+  </joint>
+  <link name="camera_link">
+    <visual>
+      <origin xyz="0 0 0" rpy="0 0 0"/>
+      <geometry>
+        <cylinder length="0.0476" radius="0.0381"/>
+      </geometry>
+      <material name="light_black"/>
+    </visual>
+    <inertial>
+      <origin xyz="0 0 0" />
+      <mass value="0.220" />
+      <inertia ixx="1.214e-4"
+               ixy="0.0" iyy="1.214e-4"
+               ixz="0.0" iyz="0.0" izz="1.597e-4" />
+    </inertial>
+  </link>
 </robot>
