Commit message: moved openrover_demo into openrover_bringup and openrover_navigation

File: openrover_description/urdf/rover.urdf (robot description, URDF)
Before this commit: robot 2WD_rover_robotics, 11 links, 10 joints
Links:
- link base_link: geometry collision box size=0.42 0.25 0.12; visual mesh filename=package://openrover_navigation/meshes/2WD_OpenRover.stl scale=1 1 1
- link caster_back_left_link: geometry collision cylinder length=0.0035 radius=0.05; visual mesh filename=package://openrover_navigation/meshes/left_caster_wheel.stl scale=1 1 1
- link caster_back_right_link: geometry collision cylinder length=0.0035 radius=0.05; visual mesh filename=package://openrover_navigation/meshes/right_caster_wheel.stl scale=1 1 1
- link sheetmetal_link: geometry collision box size=0.065 0.4 0.008; visual mesh filename=package://openrover_navigation/meshes/sheetmetal_part.stl scale=1 1 1
- link wheel_left_link: geometry collision cylinder length=0.07 radius=0.12; visual mesh filename=package://openrover_navigation/meshes/left_wheel.stl scale=1 1 1
- link wheel_right_link: geometry collision cylinder length=0.07 radius=0.12; visual mesh filename=package://openrover_navigation/meshes/right_wheel.stl scale=1 1 1

File: openrover_description/urdf/rover.urdf.xacro (robot description, xacro)
@@ -1,6 +1,6 @@
 <?xml version="1.0" ?>
 <robot name="2WD_rover_robotics" xmlns:xacro="http://ros.org/wiki/xacro">
-  <xacro:include filename="$(find openrover_demo)/urdf/common_properties.xacro"/>
-  <xacro:include filename="$(find openrover_demo)/urdf/2WD_Rover.gazebo.xacro"/>
+  <xacro:include filename="$(find openrover_navigation)/urdf/common_properties.xacro"/>
+  <xacro:include filename="$(find openrover_navigation)/urdf/2WD_Rover.gazebo.xacro"/>
   <link name="base_footprint"/>
   <joint name="base_joint" type="fixed">
@@ -13,5 +13,5 @@
       <origin xyz="-0.142 0 0.055" rpy="0 0 1.57"/>
       <geometry>
-        <mesh filename="package://openrover_demo/meshes/2WD_OpenRover.stl" scale="1 1 1"/>
+        <mesh filename="package://openrover_navigation/meshes/2WD_OpenRover.stl" scale="1 1 1"/>
       <!--
       <origin xyz="-0.142 0 0" rpy="0 0 0"/>
@@ -46,5 +46,5 @@
       <origin xyz="0 0 0" rpy="-1.57 0 0"/>
       <geometry>
-        <mesh filename="package://openrover_demo/meshes/left_wheel.stl" scale="1 1 1"/>
+        <mesh filename="package://openrover_navigation/meshes/left_wheel.stl" scale="1 1 1"/>
       <!--
       <origin xyz="0 0 0" rpy="0 0 3.14"/>
@@ -79,5 +79,5 @@
       <origin xyz="0 0 0" rpy="1.57 0 0"/>
       <geometry>
-        <mesh filename="package://openrover_demo/meshes/right_wheel.stl" scale="1 1 1"/>
+        <mesh filename="package://openrover_navigation/meshes/right_wheel.stl" scale="1 1 1"/>
       <!--
       <origin xyz="0 0 0" rpy="0 0 0"/>
@@ -111,5 +111,5 @@
       <origin xyz="0 0 0" rpy="1.57 0 -1.57"/>
       <geometry>
-        <mesh filename="package://openrover_demo/meshes/sheetmetal_part.stl" scale="1 1 1"/>
+        <mesh filename="package://openrover_navigation/meshes/sheetmetal_part.stl" scale="1 1 1"/>
       <!--
       <origin xyz="0 0 0" rpy="0 0 0"/>
@@ -229,5 +229,5 @@
       <origin xyz="0 0 0" rpy="1.57 0 3.14"/>
       <geometry>
-        <mesh filename="package://openrover_demo/meshes/left_caster_wheel.stl" scale="1 1 1"/>
+        <mesh filename="package://openrover_navigation/meshes/left_caster_wheel.stl" scale="1 1 1"/>
       <!--
       <origin xyz="-0.028 0 -0.065" rpy="1.57 0 3.14"/>
@@ -263,5 +263,5 @@
       <origin xyz="0 0 0" rpy="1.57 0 3.14"/>
       <geometry>
-        <mesh filename="package://openrover_demo/meshes/right_caster_wheel.stl" scale="1 1 1"/>
+        <mesh filename="package://openrover_navigation/meshes/right_caster_wheel.stl" scale="1 1 1"/>
       <!--
       <origin xyz="-0.028 0 -0.065" rpy="1.57 0 3.14"/>
