Commit message: added support for gazebo simulation

File: rover_description/urdf/2WD_Rover.gazebo.xacro (robot description, xacro)
@@ -2,7 +2,4 @@
 <robot name="rover_sim" xmlns:xacro="http://ros.org/wiki/xacro">
   <gazebo reference="base_link">
-    <material>Gazebo/FlatBlack</material>
-  </gazebo>
-  <gazebo reference="sheetmetal_link">
     <material>Gazebo/FlatBlack</material>
   </gazebo>

File: rover_description/urdf/rover.urdf (robot description, URDF)
Before this commit: robot 2WD_rover_robotics, 11 links, 10 joints
Links:
- removed link sheetmetal_link
- link base_link: geometry collision box size=0.42 0.25 0.12; visual mesh filename=package://rover_description/meshes/2WD_Rover.stl scale=0.001 0.001 0.001
Joints:
- removed joint sheetmetal_joint
- joint caster_back_left_joint: origin xyz=-0.01 0.17 -0.01 rpy=0 0 0 -> xyz=-0.354 0.1715 -0.01 rpy=0 0 0; parent sheetmetal_link -> base_link
- joint caster_back_right_joint: origin xyz=-0.01 -0.17 -0.01 rpy=0 0 0 -> xyz=-0.354 -0.1685 -0.01 rpy=0 0 0; parent sheetmetal_link -> base_link

File: rover_description/urdf/rover.urdf.xacro (robot description, xacro)
@@ -11,7 +11,7 @@
   <link name="base_link">
     <visual>
-      <origin xyz="-0.142 0 0.055" rpy="0 0 1.57"/>
-      <geometry>
-        <mesh filename="package://rover_description/meshes/2WD_rover.stl" scale="1 1 1"/>
+      <origin xyz="0 0 0" rpy="1.57 0 1.57"/>
+      <geometry>
+        <mesh filename="package://rover_description/meshes/2WD_Rover.stl" scale="0.001 0.001 0.001"/>
       <!--
       <origin xyz="-0.142 0 0" rpy="0 0 0"/>
@@ -102,36 +102,4 @@
     </inertial>
   </link>
-  <joint name="sheetmetal_joint" type="fixed">
-    <parent link="base_link"/>
-    <child link="sheetmetal_link"/>
-    <origin xyz="-0.35 0 0" rpy="0 0 0"/>
-  </joint>
-  <link name="sheetmetal_link">
-    <visual>
-      <origin xyz="0 0 0" rpy="1.57 0 -1.57"/>
-      <geometry>
-        <mesh filename="package://rover_description/meshes/sheetmetal_part.stl" scale="1 1 1"/>
-      <!--
-      <origin xyz="0 0 0" rpy="0 0 0"/>
-      <geometry>
-        <box size="0.065 0.4 0.008"/>
-        -->
-      </geometry>
-      <material name="dark"/>
-    </visual>
-    <collision>
-      <origin xyz="-0.007 0 0" rpy="0 0 0"/>
-      <geometry>
-        <box size="0.065 0.4 0.008"/>
-      </geometry>
-    </collision>
-    <inertial>
-      <origin xyz="0 0 0" />
-      <mass value="0.6" />
-      <inertia ixx="8.020e-3"
-               ixy="0.0" iyy="2.313e-4"
-               ixz="0.0" iyz="0.0" izz="8.211e-3" />
-    </inertial>
-  </link>
   <joint name="plate_link_joint" type="fixed">
     <parent link="base_link"/>
@@ -219,7 +187,7 @@
   </link>
   <joint name="caster_back_left_joint" type="continuous">
-    <parent link="sheetmetal_link"/>
+    <parent link="base_link"/>
     <child link="caster_back_left_link"/>
-    <origin xyz="-0.01 0.17 -0.01" rpy="0 0 0"/>
+    <origin xyz="-0.354 0.1715 -0.01" rpy="0 0 0"/>
     <axis xyz="0 0 1"/>
     <dynamics damping="0.1" friction="0.01"/>
@@ -253,7 +221,7 @@
   </link>
   <joint name="caster_back_right_joint" type="continuous">
-    <parent link="sheetmetal_link"/>
+    <parent link="base_link"/>
     <child link="caster_back_right_link"/>
-    <origin xyz="-0.01 -0.17 -0.01" rpy="0 0 0"/>
+    <origin xyz="-0.354 -0.1685 -0.01" rpy="0 0 0"/>
     <axis xyz="0 0 1"/>
     <dynamics damping="0.1" friction="0.01"/>
