Commit message: nickp final waypoint

File: rover_description/urdf/rover.urdf (robot description, URDF)
Before this commit: robot 2WD_rover_robotics, 10 links, 9 joints
Joints:
- joint imu_link_joint: origin xyz=0.1365 0 0.0026 rpy=0 0 0 -> xyz=-0.0032 0 0.0 rpy=0 0 0
- joint lidar_link_joint: origin xyz=0.10795 0 0.0635 rpy=0 0 3.14 -> xyz=0.202 0 0.0635 rpy=0 0 3.14

File: rover_description/urdf/rover.urdf.xacro (robot description, xacro)
@@ -126,5 +126,5 @@
     <parent link="plate_link"/>
     <child link="imu_link"/>
-    <origin xyz="0.1365 0 0.0026" rpy="0 0 0"/>
+    <origin xyz="-0.0032 0 0.0" rpy="0 0 0"/>
   </joint>
   <link name="imu_link">
@@ -168,5 +168,5 @@
     <parent link="cpu_link"/>
     <child link="lidar_link"/>
-    <origin xyz="0.10795 0 0.0635" rpy="0 0 3.14"/>
+    <origin xyz="0.202 0 0.0635" rpy="0 0 3.14"/>
   </joint>
   <link name="lidar_link">
